File: Kicad/CurrentFeedbackAmp/CurrentFeedbackAmp.kicad_pcb (KiCad board)
At the start: 2 copper layers, 200 x 100 mm, 93 parts, among them J1 Vin, J10 Protecc_Sup_In1, J11 Protecc_Inf_In1, J12 Protecc_Sup_In2, J13 Vdd, J14 Vcc, J15 Masa Filtros, J16 Masa Bornera Carga, J17 Bornera Carga, J2 Test_Realim_Out, J3 Masa etapa inicial, J4 Protecc_Sup_Out, J5 Protecc_Inf_Out, J6 VccTL, J7 VddTL, J8 Test_Etapa_3_Inf, J9 Test_Etapa_3_Sup, Q1 TIP42C, Q13 BC559, Q14 BC559, Q15 BC559, Q16 BC549, Q17 BC549, Q18 BC549, Q19 BC559, Q20 BC549, Q21 BC559, Q22 BC549, Q24 BD136, Q33 BD135, Q34 TIP41C, Q35 BC559, Q36 BC549, Q37 BC549, Q38 BC549, Q39 BC549, Q40 BC559, Q41 BC559, Q42 BC559, T1 BC548, T2 BC548, U2 TL082

Commit message: algunas pistas
Parts:
- moved C4 32.4 mm to (192.4, 92.7), turned to 270 degrees
- moved R32.1 30.9 mm to (114.9, 109.9), turned to 270 degrees
- moved Q1 30.5 mm to (234.3, 114.9), turned to 270 degrees
- moved C3 29.4 mm to (102.2, 99.1), turned to 90 degrees
- moved Rref3 28.3 mm to (243.8, 64.8), turned to 0 degrees
- moved R31.2 27.4 mm to (199.4, 110.5), turned to 270 degrees
- moved J11 26.1 mm to (94.0, 125.1), turned to 90 degrees
- moved R32.3 22.0 mm to (108.6, 109.9), turned to 270 degrees
- moved C1 20.7 mm to (176.5, 121.9)
- moved R31.3 20.1 mm to (193.0, 125.7), turned to 90 degrees
- moved Q34 18.5 mm to (83.2, 120.0), turned to 90 degrees
- moved J9 17.6 mm to (205.7, 90.8)
- moved C5 15.9 mm to (151.1, 85.7)
- moved C6 15.9 mm to (132.2, 77.5)
- moved R15 15.9 mm to (142.9, 85.1)
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Routing:
- net Net-(Q1-Pad1): track 0.00 -> 58.9 mm
- net Net-(Q24-Pad2): track 0.00 -> 41.9 mm
- net Net-(C9-Pad2): track 0.00 -> 39.1 mm
- net Net-(J11-Pad1): track 0.00 -> 34.9 mm
- net DC.servo.Input: track 0.00 -> 12.7 mm
- net Net-(Q36-Pad1): track 0.00 -> 8.25 mm
Other:
- net class Corriente 2.2A added: clearance 0.2, trace_width 0.75, via_dia 0.6, via_drill 0.4
