File: Kicad/CurrentFeedbackAmp/CurrentFeedbackAmp.sch (KiCad schematic (older format))
At the start: 25 parts

Commit message: Circuito casi completo en kicad y testeo de proteccion con foldback
Parts:
- removed Q? (x3): Q_NPN_BEC, symbol CurrentFeedbackAmp-rescue:Q_NPN_BEC-device
- removed R? (x3): R, symbol pspice:R
- added C? (x2): CP, symbol CP
- added C? (x10): C, symbol C
- added J? (x14): Conn_01x01, symbol Conn_01x01
- added Q? (x9): BC559, TO_SOT_Packages_THT:TO-92_Molded_Narrow, symbol BC559
- added Q?: Q_NPN_BEC, symbol CurrentFeedbackAmp-rescue:Q_NPN_BEC-device
- added Q? (x8): BC549, TO_SOT_Packages_THT:TO-92_Molded_Narrow, symbol BC549
- added Q? (x2): BC548, TO_SOT_Packages_THT:TO-92_Molded_Narrow, symbol BC548
- added Q?: BD135, TO_SOT_Packages_THT:TO-126_Vertical, symbol BD135
- added Q?: TIP42C, TO_SOT_Packages_THT:TO-220_Vertical, symbol TIP42C
- added Q?: BD136, TO_SOT_Packages_THT:TO-126_Vertical, symbol BD136
- added Q?: TIP41C, TO_SOT_Packages_THT:TO-220_Vertical, symbol TIP41C
- added R? (x9): R, symbol pspice:R
- added RV? (x3): POT, symbol POT
- added U?: TL082, symbol TL082
Connections:
- net labels added: DC.servo.Input, DC.servo.Output, GND
- wire segments 8 -> 126
- no-connect marks 0 -> 1

Commit message: Va el esquematico de KiCAD con nombres y numeros
Parts:
- gave numbers to parts that had none: 82

Commit message: va el esquematico incluyendo las resistencias de potencia
Parts:
- removed Q39: Q_NPN_BEC, symbol CurrentFeedbackAmp-rescue:Q_NPN_BEC-device
- added Q39: BC549, TO_SOT_Packages_THT:TO-92_Molded_Narrow, symbol BC549
- added R31.1, R31.2, R32.1, R32.2: R, symbol pspice:R
- renumbered R31 to R31.3, R32 to R32.3
Connections:
- wire segments 126 -> 130
Changed lines of the file:
@@
 $EndComp
 $Comp
-L GND #PWR?
+L GND #PWR01
 U 1 1 5B29B1BA
 P 3400 4300
-F 0 "#PWR?" H 3400 4050 50  0001 C CNN
+F 0 "#PWR01" H 3400 4050 50  0001 C CNN
 F 1 "GND" H 3400 4150 50  0000 C CNN
 F 2 "" H 3400 4300 50  0001 C CNN
@@
 $EndComp
 $Comp
-L GND #PWR?
+L GND #PWR02
 U 1 1 5B29E717
 P 3400 3650
-F 0 "#PWR?" H 3400 3400 50  0001 C CNN
+F 0 "#PWR02" H 3400 3400 50  0001 C CNN
 F 1 "GND" H 3400 3500 50  0000 C CNN
 F 2 "" H 3400 3650 50  0001 C CNN
@@
 $EndComp
 $Comp
-L CurrentFeedbackAmp-rescue:Q_NPN_BEC-device Q39
-U 1 1 5B2A0D60
-P 4200 3100
-F 0 "Q39" H 4391 3146 50  0000 L CNN
-F 1 "Q_NPN_BEC" H 4391 3055 50  0000 L CNN
-F 2 "" H 4400 3200 50  0000 C CNN
-F 3 "" H 4200 3100 50  0000 C CNN
-	1    4200 3100
-	1    0    0    -1
-$EndComp
-$Comp
 L pspice:R R30
 U 1 1 5B2A2501
@@
 $EndComp
 $Comp
-L GND #PWR?
+L GND #PWR03
 U 1 1 5B2A2B9D
 P 4100 1000
-F 0 "#PWR?" H 4100 750 50  0001 C CNN
+F 0 "#PWR03" H 4100 750 50  0001 C CNN
 F 1 "GND" H 4100 850 50  0000 C CNN
 F 2 "" H 4100 1000 50  0001 C CNN
@@
 $EndComp
 $Comp
-L GND #PWR?
+L GND #PWR04
 U 1 1 5B2A3C91
 P 4100 6200
-F 0 "#PWR?" H 4100 5950 50  0001 C CNN
+F 0 "#PWR04" H 4100 5950 50  0001 C CNN
 F 1 "GND" H 4100 6050 50  0000 C CNN
 F 2 "" H 4100 6200 50  0001 C CNN
@@
 $EndComp
 $Comp
-L GND #PWR?
+L GND #PWR05
 U 1 1 5B2B9157
 P 10850 2100
-F 0 "#PWR?" H 10850 1850 50  0001 C CNN
+F 0 "#PWR05" H 10850 1850 50  0001 C CNN
 F 1 "GND" H 10850 1950 50  0000 C CNN
 F 2 "" H 10850 2100 50  0001 C CNN
@@
 $EndComp
 $Comp
-L pspice:R R31
+L pspice:R R31.3
 U 1 1 5B1B0CB2
 P 10350 3350
-F 0 "R31" H 10418 3396 50  0000 L CNN
+F 0 "R31.3" H 10418 3396 50  0000 L CNN
 F 1 "R" H 10418 3305 50  0000 L CNN
 F 2 "" H 10350 3350 50  0001 C CNN
@@
 $EndComp
 $Comp
-L pspice:R R32
+L pspice:R R32.3
 U 1 1 5B1B0B5C
 P 10350 3950
-F 0 "R32" H 10418 3996 50  0000 L CNN
+F 0 "R32.3" H 10418 3996 50  0000 L CNN
 F 1 "R" H 10418 3905 50  0000 L CNN
 F 2 "" H 10350 3950 50  0001 C CNN
@@
 $EndComp
 $Comp
-L GND #PWR?
+L GND #PWR06
 U 1 1 5B2C4D91
 P 10900 5100
-F 0 "#PWR?" H 10900 4850 50  0001 C CNN
+F 0 "#PWR06" H 10900 4850 50  0001 C CNN
 F 1 "GND" H 10900 4950 50  0000 C CNN
 F 2 "" H 10900 5100 50  0001 C CNN
@@
 $EndComp
 $Comp
-L GND #PWR?
+L GND #PWR07
 U 1 1 5B2CE6CA
 P 5600 7100
-F 0 "#PWR?" H 5600 6850 50  0001 C CNN
+F 0 "#PWR07" H 5600 6850 50  0001 C CNN
 F 1 "GND" H 5600 6950 50  0000 C CNN
 F 2 "" H 5600 7100 50  0001 C CNN
@@
 $EndComp
 $Comp
-L GND #PWR?
+L GND #PWR08
 U 1 1 5B2CEB9C
 P 4500 7250
-F 0 "#PWR?" H 4500 7000 50  0001 C CNN
+F 0 "#PWR08" H 4500 7000 50  0001 C CNN
 F 1 "GND" H 4500 7100 50  0000 C CNN
 F 2 "" H 4500 7250 50  0001 C CNN
@@
 $EndComp
 $Comp
-L GND #PWR?
+L GND #PWR09
 U 1 1 5B2CF9A4
 P 4350 8050
-F 0 "#PWR?" H 4350 7800 50  0001 C CNN
+F 0 "#PWR09" H 4350 7800 50  0001 C CNN
 F 1 "GND" H 4350 7900 50  0000 C CNN
 F 2 "" H 4350 8050 50  0001 C CNN
@@
 	10350 3600 10350 3700
 Wire Wire Line
-	6550 4050 9950 4050
-Wire Wire Line
-	9950 4050 9950 3650
-Wire Wire Line
-	9950 3650 11150 3650
+	9450 3650 11150 3650
 Connection ~ 10350 2800
 Connection ~ 10350 4500
@@
 	2400 4350 2250 4350
 NoConn ~ 2250 4250
+$Comp
+L BC549 Q39
+U 1 1 5B2BE4CF
+P 4200 3100
+F 0 "Q39" H 4400 3175 50  0000 L CNN
+F 1 "BC549" H 4400 3100 50  0000 L CNN
+F 2 "TO_SOT_Packages_THT:TO-92_Molded_Narrow" H 4400 3025 50  0001 L CIN
+F 3 "" H 4200 3100 50  0001 L CNN
+	1    4200 3100
+	1    0    0    -1
+$EndComp
+$Comp
+L pspice:R R31.2
+U 1 1 5B2BFA26
+P 10150 3350
+F 0 "R31.2" H 10218 3396 50  0000 L CNN
+F 1 "R" H 10218 3305 50  0000 L CNN
+F 2 "" H 10150 3350 50  0001 C CNN
+F 3 "" H 10150 3350 50  0001 C CNN
+	1    10150 3350
+	1    0    0    -1
+$EndComp
+$Comp
+L pspice:R R31.1
+U 1 1 5B2BFB33
+P 9950 3350
+F 0 "R31.1" H 10018 3396 50  0000 L CNN
+F 1 "R" H 10018 3305 50  0000 L CNN
+F 2 "" H 9950 3350 50  0001 C CNN
+F 3 "" H 9950 3350 50  0001 C CNN
+	1    9950 3350
+	1    0    0    -1
+$EndComp
+$Comp
+L pspice:R R32.2
+U 1 1 5B2BFC9F
+P 10150 3950
+F 0 "R32.2" H 10218 3996 50  0000 L CNN
+F 1 "R" H 10218 3905 50  0000 L CNN
+F 2 "" H 10150 3950 50  0001 C CNN
+F 3 "" H 10150 3950 50  0001 C CNN
+	1    10150 3950
+	1    0    0    -1
+$EndComp
+$Comp
+L pspice:R R32.1
+U 1 1 5B2BFE0B
+P 9950 3950
+F 0 "R32.1" H 10018 3996 50  0000 L CNN
+F 1 "R" H 10018 3905 50  0000 L CNN
+F 2 "" H 9950 3950 50  0001 C CNN
+F 3 "" H 9950 3950 50  0001 C CNN
+	1    9950 3950
+	1    0    0    -1
+$EndComp
+Wire Wire Line
+	10150 3700 10150 3600
+Wire Wire Line
+	9950 3700 9950 3600
+Connection ~ 10150 3650
+Connection ~ 9950 3650
+Wire Wire Line
+	9950 4200 10350 4200
+Wire Wire Line
+	10350 3100 9950 3100
+Connection ~ 10150 3100
+Connection ~ 10150 4200
+Wire Wire Line
+	9450 3650 9450 4050
+Wire Wire Line
+	9450 4050 6550 4050
 $EndSCHEMATC

Commit message: Casi todos los componentes con su respectivo modelo asociado
Parts:
- C1, C11, C12, C2, C3, C4, C5, C6, C8, C9: footprint (none) -> Capacitors_THT:C_Disc_D5.0mm_W2.5mm_P5.00mm
- C10, C7: footprint (none) -> Capacitors_THT:CP_Radial_D5.0mm_P2.50mm
- J1, J10, J11, J12, J13, J14, J2, J3, J4, J5, J6, J7, J8, J9: footprint (none) -> Connectors:1pin
- Q13, Q14, Q15, Q16, Q17, Q18, Q19, Q20, Q21, Q22, Q35, Q36, Q37, Q38, Q39, Q40, Q41, Q42, T1, T2: footprint TO_SOT_Packages_THT:TO-92_Molded_Narrow -> TO_SOT_Packages_THT:TO-92_Inline_Narrow_Oval
- R1, R10, R11, R13, R14, R15, R16, R17, R18, R19, R2, R20, R21, R22, R23, R24, R25, R26, R27, R3, R30, R4, R5, R6, R8, R9: footprint (none) -> Resistors_SMD:R_0805_HandSoldering
- R31.1, R31.2, R31.3, R32.1, R32.2, R32.3: footprint (none) -> Resistors_THT:R_Axial_DIN0414_L11.9mm_D4.5mm_P15.24mm_Horizontal
- Rref1, Rref2: footprint (none) -> Potentiometers:Potentiometer_Trimmer_Bourns_3266Y
- Rref3: footprint (none) -> Potentiometers:Potentiometer_Alps_RK163_Single_Vertical
- U2: footprint (none) -> SMD_Packages:SOIC-8-N
Connections:
- wire segments 130 -> 129

Commit message: Ahora el PCB tiene agujeros para montar la placa y modifique el modelo de los pines
Parts:
- added MK1, MK2, MK3, MK4: Mounting_Hole, Mounting_Holes:MountingHole_2.2mm_M2, symbol Mounting_Hole
- J1, J10, J11, J12, J13, J14, J2, J3, J4, J5, J6, J7, J8, J9: footprint Connectors:1pin -> Connectors:PINTST
Changed lines of the file:
@@
 LIBS:zetex
 LIBS:Zilog
-LIBS:ECA-1HM101
 LIBS:CurrentFeedbackAmp-cache
 EELAYER 25 0
@@
 F 0 "J1" H 3400 4050 50  0000 C CNN
 F 1 "Conn_01x01" H 3400 3850 50  0000 C CNN
-F 2 "Connectors:1pin" H 3400 3950 50  0001 C CNN
+F 2 "Connectors:PINTST" H 3400 3950 50  0001 C CNN
 F 3 "" H 3400 3950 50  0001 C CNN
 	1    3400 3950
@@
 F 0 "J2" H 2300 7750 50  0000 C CNN
 F 1 "Conn_01x01" H 2300 7550 50  0000 C CNN
-F 2 "Connectors:1pin" H 2300 7650 50  0001 C CNN
+F 2 "Connectors:PINTST" H 2300 7650 50  0001 C CNN
 F 3 "" H 2300 7650 50  0001 C CNN
 	1    2300 7650
@@
 F 0 "J3" H 10900 3950 50  0000 C CNN
 F 1 "Conn_01x01" H 10900 3750 50  0000 C CNN
-F 2 "Connectors:1pin" H 10900 3850 50  0001 C CNN
+F 2 "Connectors:PINTST" H 10900 3850 50  0001 C CNN
 F 3 "" H 10900 3850 50  0001 C CNN
 	1    10900 3850
@@
 F 0 "J10" H 10700 2900 50  0000 C CNN
 F 1 "Conn_01x01" H 10700 2700 50  0000 C CNN
-F 2 "Connectors:1pin" H 10700 2800 50  0001 C CNN
+F 2 "Connectors:PINTST" H 10700 2800 50  0001 C CNN
 F 3 "" H 10700 2800 50  0001 C CNN
 	1    10700 2800
@@
 F 0 "J11" H 10700 4600 50  0000 C CNN
 F 1 "Conn_01x01" H 10700 4400 50  0000 C CNN
-F 2 "Connectors:1pin" H 10700 4500 50  0001 C CNN
+F 2 "Connectors:PINTST" H 10700 4500 50  0001 C CNN
 F 3 "" H 10700 4500 50  0001 C CNN
 	1    10700 4500
@@
 F 0 "J4" H 3100 3200 50  0000 C CNN
 F 1 "Conn_01x01" H 3100 3000 50  0000 C CNN
-F 2 "Connectors:1pin" H 3100 3100 50  0001 C CNN
+F 2 "Connectors:PINTST" H 3100 3100 50  0001 C CNN
 F 3 "" H 3100 3100 50  0001 C CNN
 	1    3100 3100
@@
 F 0 "J5" H 3050 4800 50  0000 C CNN
 F 1 "Conn_01x01" H 3050 4600 50  0000 C CNN
-F 2 "Connectors:1pin" H 3050 4700 50  0001 C CNN
+F 2 "Connectors:PINTST" H 3050 4700 50  0001 C CNN
 F 3 "" H 3050 4700 50  0001 C CNN
 	1    3050 4700
@@
 F 0 "J14" H 11250 1700 50  0000 C CNN
 F 1 "Conn_01x01" H 11250 1500 50  0000 C CNN
-F 2 "Connectors:1pin" H 11250 1600 50  0001 C CNN
+F 2 "Connectors:PINTST" H 11250 1600 50  0001 C CNN
 F 3 "" H 11250 1600 50  0001 C CNN
 	1    11250 1600
@@
 F 0 "J13" H 11250 5700 50  0000 C CNN
 F 1 "Conn_01x01" H 11250 5500 50  0000 C CNN
-F 2 "Connectors:1pin" H 11250 5600 50  0001 C CNN
+F 2 "Connectors:PINTST" H 11250 5600 50  0001 C CNN
 F 3 "" H 11250 5600 50  0001 C CNN
 	1    11250 5600
@@
 F 0 "J9" H 8450 2700 50  0000 C CNN
 F 1 "Conn_01x01" H 8450 2500 50  0000 C CNN
-F 2 "Connectors:1pin" H 8450 2600 50  0001 C CNN
+F 2 "Connectors:PINTST" H 8450 2600 50  0001 C CNN
 F 3 "" H 8450 2600 50  0001 C CNN
 	1    8450 2600
@@
 F 0 "J8" H 7450 4800 50  0000 C CNN
 F 1 "Conn_01x01" H 7450 4600 50  0000 C CNN
-F 2 "Connectors:1pin" H 7450 4700 50  0001 C CNN
+F 2 "Connectors:PINTST" H 7450 4700 50  0001 C CNN
 F 3 "" H 7450 4700 50  0001 C CNN
 	1    7450 4700
@@
 F 0 "J7" H 3500 8050 50  0000 C CNN
 F 1 "Conn_01x01" H 3500 7850 50  0000 C CNN
-F 2 "Connectors:1pin" H 3500 7950 50  0001 C CNN
+F 2 "Connectors:PINTST" H 3500 7950 50  0001 C CNN
 F 3 "" H 3500 7950 50  0001 C CNN
 	1    3500 7950
@@
 F 0 "J6" H 3300 7150 50  0000 C CNN
 F 1 "Conn_01x01" H 3300 6950 50  0000 C CNN
-F 2 "Connectors:1pin" H 3300 7050 50  0001 C CNN
+F 2 "Connectors:PINTST" H 3300 7050 50  0001 C CNN
 F 3 "" H 3300 7050 50  0001 C CNN
 	1    3300 7050
@@
 F 0 "J12" H 10600 3950 50  0000 C CNN
 F 1 "Conn_01x01" H 10600 3750 50  0000 C CNN
-F 2 "Connectors:1pin" H 10600 3850 50  0001 C CNN
+F 2 "Connectors:PINTST" H 10600 3850 50  0001 C CNN
 F 3 "" H 10600 3850 50  0001 C CNN
 	1    10600 3850
@@
 Wire Wire Line
 	9450 4050 6550 4050
+$Comp
+L Mounting_Hole MK1
+U 1 1 5B2B538A
+P 1750 950
+F 0 "MK1" H 1750 1150 50  0000 C CNN
+F 1 "Mounting_Hole" H 1750 1075 50  0000 C CNN
+F 2 "Mounting_Holes:MountingHole_2.2mm_M2" H 1750 950 50  0001 C CNN
+F 3 "" H 1750 950 50  0001 C CNN
+	1    1750 950
+	1    0    0    -1
+$EndComp
+$Comp
+L Mounting_Hole MK3
+U 1 1 5B2B5586
+P 2150 950
+F 0 "MK3" H 2150 1150 50  0000 C CNN
+F 1 "Mounting_Hole" H 2150 1075 50  0000 C CNN
+F 2 "Mounting_Holes:MountingHole_2.2mm_M2" H 2150 950 50  0001 C CNN
+F 3 "" H 2150 950 50  0001 C CNN
+	1    2150 950
+	1    0    0    -1
+$EndComp
+$Comp
+L Mounting_Hole MK2
+U 1 1 5B2B56E2
+P 1750 1200
+F 0 "MK2" H 1750 1400 50  0000 C CNN
+F 1 "Mounting_Hole" H 1750 1325 50  0000 C CNN
+F 2 "Mounting_Holes:MountingHole_2.2mm_M2" H 1750 1200 50  0001 C CNN
+F 3 "" H 1750 1200 50  0001 C CNN
+	1    1750 1200
+	1    0    0    -1
+$EndComp
+$Comp
+L Mounting_Hole MK4
+U 1 1 5B2B5803
+P 2150 1200
+F 0 "MK4" H 2150 1400 50  0000 C CNN
+F 1 "Mounting_Hole" H 2150 1325 50  0000 C CNN
+F 2 "Mounting_Holes:MountingHole_2.2mm_M2" H 2150 1200 50  0001 C CNN
+F 3 "" H 2150 1200 50  0001 C CNN
+	1    2150 1200
+	1    0    0    -1
+$EndComp
 $EndSCHEMATC

Commit message: PCB: Bornera, tierras y nombre a los pines
Parts:
- added J15: Masa Filtros, Connectors:PINTST, symbol Conn_01x01
- added J16: Masa Bornera Carga, Connectors:PINTST, symbol Conn_01x01
- added J17: Bornera Carga, Connectors_Terminal_Blocks:TerminalBlock_Pheonix_MKDS1.5-2pol, symbol Screw_Terminal_01x02
- J1: value Conn_01x01 -> Vin
- J10: value Conn_01x01 -> Protecc_Sup_In1
- J11: value Conn_01x01 -> Protecc_Inf_In1
- J12: value Conn_01x01 -> Protecc_Sup_In2
- J13: value Conn_01x01 -> Vdd
- J14: value Conn_01x01 -> Vcc
- J2: value Conn_01x01 -> Test_Realim_Out
- J3: value Conn_01x01 -> Masa etapa inicial
- J4: value Conn_01x01 -> Protecc_Sup_Out
- J5: value Conn_01x01 -> Protecc_Inf_Out
- J6: value Conn_01x01 -> VccTL
- J7: value Conn_01x01 -> VddTL
- J8: value Conn_01x01 -> Test_Etapa_3_Inf
- J9: value Conn_01x01 -> Test_Etapa_3_Sup
Connections:
- wire segments 129 -> 133
Changed lines of the file:
@@
 P 3400 3950
 F 0 "J1" H 3400 4050 50  0000 C CNN
-F 1 "Conn_01x01" H 3400 3850 50  0000 C CNN
+F 1 "Vin" H 3400 3850 50  0000 C CNN
 F 2 "Connectors:PINTST" H 3400 3950 50  0001 C CNN
 F 3 "" H 3400 3950 50  0001 C CNN
@@
 P 2300 7650
 F 0 "J2" H 2300 7750 50  0000 C CNN
-F 1 "Conn_01x01" H 2300 7550 50  0000 C CNN
+F 1 "Test_Realim_Out" H 2300 7550 50  0000 C CNN
 F 2 "Connectors:PINTST" H 2300 7650 50  0001 C CNN
 F 3 "" H 2300 7650 50  0001 C CNN
@@
 $EndComp
 $Comp
-L Conn_01x01 J3
-U 1 1 5B2C837C
-P 10900 3850
-F 0 "J3" H 10900 3950 50  0000 C CNN
-F 1 "Conn_01x01" H 10900 3750 50  0000 C CNN
-F 2 "Connectors:PINTST" H 10900 3850 50  0001 C CNN
-F 3 "" H 10900 3850 50  0001 C CNN
-	1    10900 3850
-	0    1    1    0
-$EndComp
-$Comp
 L Conn_01x01 J10
 U 1 1 5B2C8E12
 P 10700 2800
 F 0 "J10" H 10700 2900 50  0000 C CNN
-F 1 "Conn_01x01" H 10700 2700 50  0000 C CNN
+F 1 "Protecc_Sup_In1" H 10700 2700 50  0000 C CNN
 F 2 "Connectors:PINTST" H 10700 2800 50  0001 C CNN
 F 3 "" H 10700 2800 50  0001 C CNN
@@
 P 10700 4500
 F 0 "J11" H 10700 4600 50  0000 C CNN
-F 1 "Conn_01x01" H 10700 4400 50  0000 C CNN
+F 1 "Protecc_Inf_In1" H 10700 4400 50  0000 C CNN
 F 2 "Connectors:PINTST" H 10700 4500 50  0001 C CNN
 F 3 "" H 10700 4500 50  0001 C CNN
@@
 P 3100 3100
 F 0 "J4" H 3100 3200 50  0000 C CNN
-F 1 "Conn_01x01" H 3100 3000 50  0000 C CNN
+F 1 "Protecc_Sup_Out" H 3100 3000 50  0000 C CNN
 F 2 "Connectors:PINTST" H 3100 3100 50  0001 C CNN
 F 3 "" H 3100 3100 50  0001 C CNN
@@
 P 3050 4700
 F 0 "J5" H 3050 4800 50  0000 C CNN
-F 1 "Conn_01x01" H 3050 4600 50  0000 C CNN
+F 1 "Protecc_Inf_Out" H 3050 4600 50  0000 C CNN
 F 2 "Connectors:PINTST" H 3050 4700 50  0001 C CNN
 F 3 "" H 3050 4700 50  0001 C CNN
@@
 P 11250 1600
 F 0 "J14" H 11250 1700 50  0000 C CNN
-F 1 "Conn_01x01" H 11250 1500 50  0000 C CNN
+F 1 "Vcc" H 11250 1500 50  0000 C CNN
 F 2 "Connectors:PINTST" H 11250 1600 50  0001 C CNN
 F 3 "" H 11250 1600 50  0001 C CNN
@@
 P 11250 5600
 F 0 "J13" H 11250 5700 50  0000 C CNN
-F 1 "Conn_01x01" H 11250 5500 50  0000 C CNN
+F 1 "Vdd" H 11250 5500 50  0000 C CNN
 F 2 "Connectors:PINTST" H 11250 5600 50  0001 C CNN
 F 3 "" H 11250 5600 50  0001 C CNN
@@
 P 8450 2600
 F 0 "J9" H 8450 2700 50  0000 C CNN
-F 1 "Conn_01x01" H 8450 2500 50  0000 C CNN
+F 1 "Test_Etapa_3_Sup" H 8450 2500 50  0000 C CNN
 F 2 "Connectors:PINTST" H 8450 2600 50  0001 C CNN
 F 3 "" H 8450 2600 50  0001 C CNN
@@
 P 7450 4700
 F 0 "J8" H 7450 4800 50  0000 C CNN
-F 1 "Conn_01x01" H 7450 4600 50  0000 C CNN
+F 1 "Test_Etapa_3_Inf" H 7450 4600 50  0000 C CNN
 F 2 "Connectors:PINTST" H 7450 4700 50  0001 C CNN
 F 3 "" H 7450 4700 50  0001 C CNN
@@
 P 3500 7950
 F 0 "J7" H 3500 8050 50  0000 C CNN
-F 1 "Conn_01x01" H 3500 7850 50  0000 C CNN
+F 1 "VddTL" H 3500 7850 50  0000 C CNN
 F 2 "Connectors:PINTST" H 3500 7950 50  0001 C CNN
 F 3 "" H 3500 7950 50  0001 C CNN
@@
 P 3300 7050
 F 0 "J6" H 3300 7150 50  0000 C CNN
-F 1 "Conn_01x01" H 3300 6950 50  0000 C CNN
+F 1 "VccTL" H 3300 6950 50  0000 C CNN
 F 2 "Connectors:PINTST" H 3300 7050 50  0001 C CNN
 F 3 "" H 3300 7050 50  0001 C CNN
@@
 P 10600 3850
 F 0 "J12" H 10600 3950 50  0000 C CNN
-F 1 "Conn_01x01" H 10600 3750 50  0000 C CNN
+F 1 "Protecc_Sup_In2" H 10600 3750 50  0000 C CNN
 F 2 "Connectors:PINTST" H 10600 3850 50  0001 C CNN
 F 3 "" H 10600 3850 50  0001 C CNN
@@
 Connection ~ 7750 1650
 Wire Wire Line
-	10350 2350 10350 3100
+	10350 3100 10350 2350
 Wire Wire Line
 	9800 2800 10500 2800
@@
 $EndComp
 Wire Wire Line
-	10150 3700 10150 3600
-Wire Wire Line
-	9950 3700 9950 3600
+	10150 3600 10150 3700
+Wire Wire Line
+	9950 3600 9950 3700
 Connection ~ 10150 3650
 Connection ~ 9950 3650
@@
 	9950 4200 10350 4200
 Wire Wire Line
-	10350 3100 9950 3100
+	9950 3100 10350 3100
 Connection ~ 10150 3100
 Connection ~ 10150 4200
@@
 	1    0    0    -1
 $EndComp
+$Comp
+L GND #PWR010
+U 1 1 5B2C1357
+P 7900 7300
+F 0 "#PWR010" H 7900 7050 50  0001 C CNN
+F 1 "GND" H 7900 7150 50  0000 C CNN
+F 2 "" H 7900 7300 50  0001 C CNN
+F 3 "" H 7900 7300 50  0001 C CNN
+	1    7900 7300
+	1    0    0    -1
+$EndComp
+$Comp
+L Conn_01x01 J3
+U 1 1 5B2C383B
+P 7900 6900
+F 0 "J3" H 7900 7000 50  0000 C CNN
+F 1 "Masa etapa inicial" H 7900 6800 50  0000 C CNN
+F 2 "Connectors:PINTST" H 7900 6900 50  0001 C CNN
+F 3 "" H 7900 6900 50  0001 C CNN
+	1    7900 6900
+	0    -1   -1   0
+$EndComp
+Wire Wire Line
+	7900 7300 7900 7100
+$Comp
+L GND #PWR011
+U 1 1 5B2CAB59
+P 8300 7300
+F 0 "#PWR011" H 8300 7050 50  0001 C CNN
+F 1 "GND" H 8300 7150 50  0000 C CNN
+F 2 "" H 8300 7300 50  0001 C CNN
+F 3 "" H 8300 7300 50  0001 C CNN
+	1    8300 7300
+	1    0    0    -1
+$EndComp
+$Comp
+L Conn_01x01 J15
+U 1 1 5B2CAB5F
+P 8300 6900
+F 0 "J15" H 8300 7000 50  0000 C CNN
+F 1 "Masa Filtros" H 8300 6800 50  0000 C CNN
+F 2 "Connectors:PINTST" H 8300 6900 50  0001 C CNN
+F 3 "" H 8300 6900 50  0001 C CNN
+	1    8300 6900
+	0    -1   -1   0
+$EndComp
+Wire Wire Line
+	8300 7300 8300 7100
+$Comp
+L Screw_Terminal_01x02 J17
+U 1 1 5B2D0185
+P 10900 3150
+F 0 "J17" H 10900 3250 50  0000 C CNN
+F 1 "Bornera Carga" H 10900 2950 50  0000 C CNN
+F 2 "Connectors_Terminal_Blocks:TerminalBlock_Pheonix_MKDS1.5-2pol" H 10900 3150 50  0001 C CNN
+F 3 "" H 10900 3150 50  0001 C CNN
+	1    10900 3150
+	0    -1   -1   0
+$EndComp
+$Comp
+L GND #PWR012
+U 1 1 5B2D146B
+P 11000 3350
+F 0 "#PWR012" H 11000 3100 50  0001 C CNN
+F 1 "GND" H 11000 3200 50  0000 C CNN
+F 2 "" H 11000 3350 50  0001 C CNN
+F 3 "" H 11000 3350 50  0001 C CNN
+	1    11000 3350
+	1    0    0    -1
+$EndComp
+Wire Wire Line
+	10900 3350 10900 3650
+$Comp
+L GND #PWR013
+U 1 1 5B2D1F1C
+P 8700 7300
+F 0 "#PWR013" H 8700 7050 50  0001 C CNN
+F 1 "GND" H 8700 7150 50  0000 C CNN
+F 2 "" H 8700 7300 50  0001 C CNN
+F 3 "" H 8700 7300 50  0001 C CNN
+	1    8700 7300
+	1    0    0    -1
+$EndComp
+$Comp
+L Conn_01x01 J16
+U 1 1 5B2D1F22
+P 8700 6900
+F 0 "J16" H 8700 7000 50  0000 C CNN
+F 1 "Masa Bornera Carga" H 8700 6800 50  0000 C CNN
+F 2 "Connectors:PINTST" H 8700 6900 50  0001 C CNN
+F 3 "" H 8700 6900 50  0001 C CNN
+	1    8700 6900
+	0    -1   -1   0
+$EndComp
+Wire Wire Line
+	8700 7300 8700 7100
 $EndSCHEMATC

Commit message: Cambio modelo de capacitores electroliticos
Parts:
- C10, C7: footprint Capacitors_THT:CP_Radial_D5.0mm_P2.50mm -> Capacitors_THT:CP_Radial_D8.0mm_P3.80mm
Changed lines of the file:
@@
 F 0 "C7" H 4125 1400 50  0000 L CNN
 F 1 "CP" H 4125 1200 50  0000 L CNN
-F 2 "Capacitors_THT:CP_Radial_D5.0mm_P2.50mm" H 4138 1150 50  0001 C CNN
+F 2 "Capacitors_THT:CP_Radial_D8.0mm_P3.80mm" H 4138 1150 50  0001 C CNN
 F 3 "" H 4100 1300 50  0001 C CNN
 	1    4100 1300
@@
 F 0 "C10" H 4125 6000 50  0000 L CNN
 F 1 "CP" H 4125 5800 50  0000 L CNN
-F 2 "Capacitors_THT:CP_Radial_D5.0mm_P2.50mm" H 4138 5750 50  0001 C CNN
+F 2 "Capacitors_THT:CP_Radial_D8.0mm_P3.80mm" H 4138 5750 50  0001 C CNN
 F 3 "" H 4100 5900 50  0001 C CNN
 	1    4100 5900
