File: Kicad/CurrentFeedbackAmp/CurrentFeedbackAmp.sch (KiCad schematic (older format))
At the start: 93 parts, among them J1 Vin, J10 Protecc_Sup_In1, J11 Protecc_Inf_In1, J12 Protecc_Sup_In2, J13 Vdd, J14 Vcc, J15 Masa Filtros, J16 Masa Bornera Carga, J17 Bornera Carga, J2 Test_Realim_Out, J3 Masa etapa inicial, J4 Protecc_Sup_Out, J5 Protecc_Inf_Out, J6 VccTL, J7 VddTL, J8 Test_Etapa_3_Inf, J9 Test_Etapa_3_Sup, Q1 TIP42C, Q13 BC559, Q14 BC559, Q15 BC559, Q16 BC549, Q17 BC549, Q18 BC549, Q19 BC559, Q20 BC549, Q21 BC559, Q22 BC549, Q24 BD136, Q33 BD135, Q34 TIP41C, Q35 BC559, Q36 BC549, Q37 BC549, Q38 BC549, Q39 BC549, Q40 BC559, Q41 BC559, Q42 BC559, T1 BC548, T2 BC548, U2 TL082

Commit message: Agregue reguiladores al kicad y complete las conexiones de los pines del tl082
Parts:
- added J18, J20, J23: Masa Reguladores, Connectors:PINTST, symbol Conn_01x01
- added J19: Vcc, Connectors:PINTST, symbol Conn_01x01
- added J21, J25, J26, J28, J29: VccTL, Connectors:PINTST, symbol Conn_01x01
- added J22: Vdd, Connectors:PINTST, symbol Conn_01x01
- added J24, J27: VddTL, Connectors:PINTST, symbol Conn_01x01
- added U1: LM7812_TO220, TO_SOT_Packages_THT:TO-220_Vertical, symbol LM7812_TO220
- added unit 2 of U2
- added U3: LM7912_TO220, TO_SOT_Packages_THT:TO-220_Vertical, symbol LM7912_TO220
Connections:
- wire segments 133 -> 135
Changed lines of the file:
@@
 Wire Wire Line
 	8700 7300 8700 7100
+$Comp
+L LM7812_TO220 U1
+U 1 1 5B2EB8FB
+P 10650 6750
+F 0 "U1" H 10500 6875 50  0000 C CNN
+F 1 "LM7812_TO220" H 10650 6875 50  0000 L CNN
+F 2 "TO_SOT_Packages_THT:TO-220_Vertical" H 10650 6975 50  0001 C CIN
+F 3 "" H 10650 6700 50  0001 C CNN
+	1    10650 6750
+	1    0    0    -1
+$EndComp
+$Comp
+L LM7912_TO220 U3
+U 1 1 5B2EBA94
+P 12200 6750
+F 0 "U3" H 12050 6625 50  0000 C CNN
+F 1 "LM7912_TO220" H 12200 6625 50  0000 L CNN
+F 2 "TO_SOT_Packages_THT:TO-220_Vertical" H 12200 6550 50  0001 C CIN
+F 3 "" H 12200 6750 50  0001 C CNN
+	1    12200 6750
+	1    0    0    1
+$EndComp
+$Comp
+L GND #PWR014
+U 1 1 5B2EDF8E
+P 9100 7300
+F 0 "#PWR014" H 9100 7050 50  0001 C CNN
+F 1 "GND" H 9100 7150 50  0000 C CNN
+F 2 "" H 9100 7300 50  0001 C CNN
+F 3 "" H 9100 7300 50  0001 C CNN
+	1    9100 7300
+	1    0    0    -1
+$EndComp
+$Comp
+L Conn_01x01 J18
+U 1 1 5B2EE0B6
+P 9100 6900
+F 0 "J18" H 9100 7000 50  0000 C CNN
+F 1 "Masa Reguladores" H 9100 6800 50  0000 C CNN
+F 2 "Connectors:PINTST" H 9100 6900 50  0001 C CNN
+F 3 "" H 9100 6900 50  0001 C CNN
+	1    9100 6900
+	0    -1   -1   0
+$EndComp
+Wire Wire Line
+	9100 7100 9100 7300
+$Comp
+L Conn_01x01 J20
+U 1 1 5B2EE562
+P 10650 7250
+F 0 "J20" H 10650 7350 50  0000 C CNN
+F 1 "Masa Reguladores" H 10650 7150 50  0000 C CNN
+F 2 "Connectors:PINTST" H 10650 7250 50  0001 C CNN
+F 3 "" H 10650 7250 50  0001 C CNN
+	1    10650 7250
+	0    1    1    0
+$EndComp
+$Comp
+L Conn_01x01 J23
+U 1 1 5B2EEBE6
+P 12200 7250
+F 0 "J23" H 12200 7350 50  0000 C CNN
+F 1 "Masa Reguladores" H 12200 7150 50  0000 C CNN
+F 2 "Connectors:PINTST" H 12200 7250 50  0001 C CNN
+F 3 "" H 12200 7250 50  0001 C CNN
+	1    12200 7250
+	0    1    1    0
+$EndComp
+$Comp
+L Conn_01x01 J19
+U 1 1 5B2F00E4
+P 10150 6750
+F 0 "J19" H 10150 6850 50  0000 C CNN
+F 1 "Vcc" H 10150 6650 50  0000 C CNN
+F 2 "Connectors:PINTST" H 10150 6750 50  0001 C CNN
+F 3 "" H 10150 6750 50  0001 C CNN
+	1    10150 6750
+	-1   0    0    1
+$EndComp
+$Comp
+L Conn_01x01 J22
+U 1 1 5B2F0327
+P 11700 6750
+F 0 "J22" H 11700 6850 50  0000 C CNN
+F 1 "Vdd" H 11700 6650 50  0000 C CNN
+F 2 "Connectors:PINTST" H 11700 6750 50  0001 C CNN
+F 3 "" H 11700 6750 50  0001 C CNN
+	1    11700 6750
+	-1   0    0    1
+$EndComp
+$Comp
+L Conn_01x01 J21
+U 1 1 5B2F0A21
+P 11150 6750
+F 0 "J21" H 11150 6850 50  0000 C CNN
+F 1 "VccTL" H 11150 6650 50  0000 C CNN
+F 2 "Connectors:PINTST" H 11150 6750 50  0001 C CNN
+F 3 "" H 11150 6750 50  0001 C CNN
+	1    11150 6750
+	1    0    0    -1
+$EndComp
+$Comp
+L Conn_01x01 J24
+U 1 1 5B2F0C98
+P 12700 6750
+F 0 "J24" H 12700 6850 50  0000 C CNN
+F 1 "VddTL" H 12700 6650 50  0000 C CNN
+F 2 "Connectors:PINTST" H 12700 6750 50  0001 C CNN
+F 3 "" H 12700 6750 50  0001 C CNN
+	1    12700 6750
+	1    0    0    -1
+$EndComp
+$Comp
+L TL082 U2
+U 2 1 5B2F3391
+P 3400 8700
+F 0 "U2" H 3400 8900 50  0000 L CNN
+F 1 "TL082" H 3400 8500 50  0000 L CNN
+F 2 "SMD_Packages:SOIC-8-N" H 3400 8700 50  0001 C CNN
+F 3 "" H 3400 8700 50  0001 C CNN
+	2    3400 8700
+	-1   0    0    1
+$EndComp
+$Comp
+L Conn_01x01 J25
+U 1 1 5B2F3703
+P 2900 8700
+F 0 "J25" H 2900 8800 50  0000 C CNN
+F 1 "VccTL" H 2900 8600 50  0000 C CNN
+F 2 "Connectors:PINTST" H 2900 8700 50  0001 C CNN
+F 3 "" H 2900 8700 50  0001 C CNN
+	1    2900 8700
+	-1   0    0    1
+$EndComp
+$Comp
+L Conn_01x01 J28
+U 1 1 5B2F38A5
+P 3900 8600
+F 0 "J28" H 3900 8700 50  0000 C CNN
+F 1 "VccTL" H 3900 8500 50  0000 C CNN
+F 2 "Connectors:PINTST" H 3900 8600 50  0001 C CNN
+F 3 "" H 3900 8600 50  0001 C CNN
+	1    3900 8600
+	1    0    0    -1
+$EndComp
+$Comp
+L Conn_01x01 J29
+U 1 1 5B2F3A1C
+P 3900 8800
+F 0 "J29" H 3900 8900 50  0000 C CNN
+F 1 "VccTL" H 3900 8700 50  0000 C CNN
+F 2 "Connectors:PINTST" H 3900 8800 50  0001 C CNN
+F 3 "" H 3900 8800 50  0001 C CNN
+	1    3900 8800
+	1    0    0    -1
+$EndComp
+$Comp
+L Conn_01x01 J26
+U 1 1 5B2F3B6E
+P 3300 8300
+F 0 "J26" H 3300 8400 50  0000 C CNN
+F 1 "VccTL" H 3300 8200 50  0000 C CNN
+F 2 "Connectors:PINTST" H 3300 8300 50  0001 C CNN
+F 3 "" H 3300 8300 50  0001 C CNN
+	1    3300 8300
+	-1   0    0    1
+$EndComp
+Wire Wire Line
+	3500 8400 3500 8300
+$Comp
+L Conn_01x01 J27
+U 1 1 5B2F3E34
+P 3500 9200
+F 0 "J27" H 3500 9300 50  0000 C CNN
+F 1 "VddTL" H 3500 9100 50  0000 C CNN
+F 2 "Connectors:PINTST" H 3500 9200 50  0001 C CNN
+F 3 "" H 3500 9200 50  0001 C CNN
+	1    3500 9200
+	0    1    1    0
+$EndComp
 $EndSCHEMATC
