File: Kicad/CurrentFeedbackAmp/CurrentFeedbackAmp.sch (KiCad schematic (older format))
At the start: 107 parts, among them J1 Vin, J10 Protecc_Sup_In1, J11 Protecc_Inf_In1, J12 Protecc_Sup_In2, J13 Vdd, J14 Vcc, J15 Masa Filtros, J16 Masa Bornera Carga, J17 Bornera Carga, J18 Masa Reguladores, J19 Vcc, J2 Test_Realim_Out, J20 Masa Reguladores, J21 VccTL, J22 Vdd, J23 Masa Reguladores, J24 VddTL, J25 VccTL, J26 VccTL, J27 VddTL, J28 VccTL, J29 VccTL, J3 Masa etapa inicial, J4 Protecc_Sup_Out, J5 Protecc_Inf_Out, J6 VccTL, J7 VddTL, J8 Test_Etapa_3_Inf, J9 Test_Etapa_3_Sup, Q1 TIP42C, Q13 BC559, Q14 BC559, Q15 BC559, Q16 BC549, Q17 BC549, Q18 BC549, Q19 BC559, Q20 BC549, Q21 BC559, Q22 BC549, Q24 BD136, Q33 BD135, Q34 TIP41C, Q35 BC559, Q36 BC549, Q37 BC549, Q38 BC549, Q39 BC549, Q40 BC559, Q41 BC559, Q42 BC559, T1 BC548, T2 BC548, U1 LM7812_TO220, U2 TL082, U3 LM7912_TO220

Commit message: Conexion correcta de pines inutilizados del TL082 y la guia que explica por que
Parts:
- removed J25, J28, J29: VccTL, Connectors:PINTST, symbol Conn_01x01
- added J?: Masa Reguladores, Connectors:PINTST, symbol Conn_01x01
Connections:
- wire segments 135 -> 140
Changed lines of the file:
@@
-$EndComp
-$Comp
-L Conn_01x01 J25
-U 1 1 5B2F3703
-P 2900 8700
-F 0 "J25" H 2900 8800 50  0000 C CNN
-F 1 "VccTL" H 2900 8600 50  0000 C CNN
-F 2 "Connectors:PINTST" H 2900 8700 50  0001 C CNN
-F 3 "" H 2900 8700 50  0001 C CNN
-	1    2900 8700
-	-1   0    0    1
-$EndComp
-$Comp
-L Conn_01x01 J28
-U 1 1 5B2F38A5
-P 3900 8600
-F 0 "J28" H 3900 8700 50  0000 C CNN
-F 1 "VccTL" H 3900 8500 50  0000 C CNN
-F 2 "Connectors:PINTST" H 3900 8600 50  0001 C CNN
-F 3 "" H 3900 8600 50  0001 C CNN
-	1    3900 8600
-	1    0    0    -1
-$EndComp
-$Comp
-L Conn_01x01 J29
-U 1 1 5B2F3A1C
-P 3900 8800
-F 0 "J29" H 3900 8900 50  0000 C CNN
-F 1 "VccTL" H 3900 8700 50  0000 C CNN
-F 2 "Connectors:PINTST" H 3900 8800 50  0001 C CNN
-F 3 "" H 3900 8800 50  0001 C CNN
-	1    3900 8800
-	1    0    0    -1
 $EndComp
 $Comp
@@
 	0    1    1    0
 $EndComp
+Wire Wire Line
+	3700 8600 4250 8600
+Wire Wire Line
+	4250 8600 4250 9400
+Wire Wire Line
+	4250 9400 3000 9400
+Wire Wire Line
+	3000 9400 3000 8700
+Wire Wire Line
+	3000 8700 3100 8700
+$Comp
+L Conn_01x01 J?
+U 1 1 5B2EBC4E
+P 3900 8800
+F 0 "J?" H 3900 8900 50  0000 C CNN
+F 1 "Masa Reguladores" H 3900 8700 50  0000 C CNN
+F 2 "Connectors:PINTST" H 3900 8800 50  0001 C CNN
+F 3 "" H 3900 8800 50  0001 C CNN
+	1    3900 8800
+	1    0    0    -1
+$EndComp
 $EndSCHEMATC

Commit message: Elimine algunos pins que no deberian ir porque van a ser conectados con pistas
Parts:
- removed J19: Vcc, Connectors:PINTST, symbol Conn_01x01
- removed J21, J26, J6: VccTL, Connectors:PINTST, symbol Conn_01x01
- removed J22: Vdd, Connectors:PINTST, symbol Conn_01x01
- removed J24, J27, J7: VddTL, Connectors:PINTST, symbol Conn_01x01
- gave numbers to parts that had none: 1
Connections:
- net labels added: Vcc, VccTL, Vdd, VddTL
Changed lines of the file:
@@
 	1    0    0    -1
-$EndComp
-$Comp
-L Conn_01x01 J7
-U 1 1 5B2D255D
-P 3500 7950
-F 0 "J7" H 3500 8050 50  0000 C CNN
-F 1 "VddTL" H 3500 7850 50  0000 C CNN
-F 2 "Connectors:PINTST" H 3500 7950 50  0001 C CNN
-F 3 "" H 3500 7950 50  0001 C CNN
-	1    3500 7950
-	0    1    1    0
-$EndComp
-$Comp
-L Conn_01x01 J6
-U 1 1 5B2D351D
-P 3300 7050
-F 0 "J6" H 3300 7150 50  0000 C CNN
-F 1 "VccTL" H 3300 6950 50  0000 C CNN
-F 2 "Connectors:PINTST" H 3300 7050 50  0001 C CNN
-F 3 "" H 3300 7050 50  0001 C CNN
-	1    3300 7050
-	-1   0    0    1
 $EndComp
 Text GLabel 2100 7450 0    60   Input ~ 0
@@
 $EndComp
 $Comp
-L Conn_01x01 J19
-U 1 1 5B2F00E4
-P 10150 6750
-F 0 "J19" H 10150 6850 50  0000 C CNN
-F 1 "Vcc" H 10150 6650 50  0000 C CNN
-F 2 "Connectors:PINTST" H 10150 6750 50  0001 C CNN
-F 3 "" H 10150 6750 50  0001 C CNN
-	1    10150 6750
-	-1   0    0    1
-$EndComp
-$Comp
-L Conn_01x01 J22
-U 1 1 5B2F0327
-P 11700 6750
-F 0 "J22" H 11700 6850 50  0000 C CNN
-F 1 "Vdd" H 11700 6650 50  0000 C CNN
-F 2 "Connectors:PINTST" H 11700 6750 50  0001 C CNN
-F 3 "" H 11700 6750 50  0001 C CNN
-	1    11700 6750
-	-1   0    0    1
-$EndComp
-$Comp
-L Conn_01x01 J21
-U 1 1 5B2F0A21
-P 11150 6750
-F 0 "J21" H 11150 6850 50  0000 C CNN
-F 1 "VccTL" H 11150 6650 50  0000 C CNN
-F 2 "Connectors:PINTST" H 11150 6750 50  0001 C CNN
-F 3 "" H 11150 6750 50  0001 C CNN
-	1    11150 6750
-	1    0    0    -1
-$EndComp
-$Comp
-L Conn_01x01 J24
-U 1 1 5B2F0C98
-P 12700 6750
-F 0 "J24" H 12700 6850 50  0000 C CNN
-F 1 "VddTL" H 12700 6650 50  0000 C CNN
-F 2 "Connectors:PINTST" H 12700 6750 50  0001 C CNN
-F 3 "" H 12700 6750 50  0001 C CNN
-	1    12700 6750
-	1    0    0    -1
-$EndComp
-$Comp
 L TL082 U2
 U 2 1 5B2F3391
@@
 	-1   0    0    1
 $EndComp
-$Comp
-L Conn_01x01 J26
-U 1 1 5B2F3B6E
-P 3300 8300
-F 0 "J26" H 3300 8400 50  0000 C CNN
-F 1 "VccTL" H 3300 8200 50  0000 C CNN
-F 2 "Connectors:PINTST" H 3300 8300 50  0001 C CNN
-F 3 "" H 3300 8300 50  0001 C CNN
-	1    3300 8300
-	-1   0    0    1
-$EndComp
 Wire Wire Line
 	3500 8400 3500 8300
-$Comp
-L Conn_01x01 J27
-U 1 1 5B2F3E34
-P 3500 9200
-F 0 "J27" H 3500 9300 50  0000 C CNN
-F 1 "VddTL" H 3500 9100 50  0000 C CNN
-F 2 "Connectors:PINTST" H 3500 9200 50  0001 C CNN
-F 3 "" H 3500 9200 50  0001 C CNN
-	1    3500 9200
-	0    1    1    0
-$EndComp
 Wire Wire Line
 	3700 8600 4250 8600
@@
 	3000 8700 3100 8700
 $Comp
-L Conn_01x01 J?
+L Conn_01x01 J25
 U 1 1 5B2EBC4E
 P 3900 8800
-F 0 "J?" H 3900 8900 50  0000 C CNN
+F 0 "J25" H 3900 8900 50  0000 C CNN
 F 1 "Masa Reguladores" H 3900 8700 50  0000 C CNN
 F 2 "Connectors:PINTST" H 3900 8800 50  0001 C CNN
@@
 	1    0    0    -1
 $EndComp
+Text GLabel 3500 9000 0    60   Input ~ 0
+VddTL
+Text GLabel 3500 7750 0    60   Input ~ 0
+VddTL
+Text GLabel 3500 8300 0    60   Input ~ 0
+VccTL
+Text GLabel 3500 7050 0    60   Input ~ 0
+VccTL
+Text GLabel 10950 6750 2    60   Input ~ 0
+VccTL
+Text GLabel 12500 6750 2    60   Input ~ 0
+VddTL
+Text GLabel 11000 1600 1    60   Input ~ 0
+Vcc
+Text GLabel 11050 5600 3    60   Input ~ 0
+Vdd
+Text GLabel 11900 6750 0    60   Input ~ 0
+Vdd
+Text GLabel 10350 6750 0    60   Input ~ 0
+Vcc
 $EndSCHEMATC

Commit message: Agregados capacitores de 1000u en sim y kicad, cambié pines de las fuentes de alimentacion por borneras, y puse valores a cada componente
Parts:
- removed J13: Vdd, Connectors:PINTST, symbol Conn_01x01
- removed J14: Vcc, Connectors:PINTST, symbol Conn_01x01
- added C13, C14: 1000u, Capacitors_THT:CP_Radial_D16.0mm_P7.50mm, symbol CP
- added J6: Bornera Vcc, Connectors_Terminal_Blocks:TerminalBlock_Pheonix_MKDS1.5-2pol, symbol Screw_Terminal_01x02
- added J7: Bornera Vdd, Connectors_Terminal_Blocks:TerminalBlock_Pheonix_MKDS1.5-2pol, symbol Screw_Terminal_01x02
- C1, C2: value C -> 10n
- C10, C7: value CP -> 100u
- C11, C12, C5, C6: value C -> 220n
- C3, C4: value C -> 10p
- C8, C9: value C -> 100n
- R1, R2: value R -> 39
- R10, R27, R30, R5: value R -> 150
- R11, R20, R21, R6: value R -> 100
- R13, R14, R25, R26: value R -> 200
- R15: value R -> 270
- R16, R17: value R -> 50
- R18: value R -> 1k
- R19: value R -> 5.1k
- R22, R23: value R -> 100k
- R24: value R -> 10k
- R3, R8: value R -> 400
- R31.1, R31.2, R31.3, R32.1, R32.2, R32.3: value R -> 1
- R4, R9: value R -> 300
Connections:
- wire segments 140 -> 144
